File: mcu.kicad_sch (KiCad schematic)
At the start: 15 parts, among them J10 Pico_Socket_B, J4 Pico_Socket_A, SW1 K3-2235D-F1, U1 MAX6816EUS+T

Commit message: Add PI3DPX1203BZLEX DisplayPort redriver and start adding it to schematic
Changed lines of the file:
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@@
 	)
 	(hierarchical_label "I2C_SCL"
-		(shape input)
+		(shape bidirectional)
 		(at 281.94 130.81 180)
 		(effects

Commit message: Wiring up DisplayPort HPD signals
Parts:
- added C88: 0.1uF, Capacitor_SMD:C_0603_1608Metric, symbol Device:C_Small
- added R32: 10k, Resistor_SMD:R_0603_1608Metric, symbol Device:R
- added TP18: TestPoint, TestPoint:TestPoint_Pad_1.0x1.0mm, symbol Connector:TestPoint
- added U19: 74LVC1G04, symbol 74xGxx:74LVC1G04
Connections:
- net GND: now also C88.1, R32.2, U19.3 (GND)
- net MUX_SEL: now also U19.2
- net VCC_3.3V: now also C88.2, U19.5 (VCC)
- new net ~{MUX_SEL}: R32.1, TP18.1, U19.4

Commit message: Start wiring up Pi Pico
Parts:
- added R30: 10k, Resistor_SMD:R_0603_1608Metric, symbol Device:R
- added R31, R33: 27, Resistor_SMD:R_0603_1608Metric, symbol Device:R
- added SW2: K3-2235D-F1, hubble:SW-TH_K3-2235D-F1, symbol Switch:SW_Push_DPDT
Connections:
- net GND: now also R30.2
- net I2C_SCL: now also A1.5 (GPIO3), J4.5 (GPIO3)
- net I2C_SDA: now also A1.4 (GPIO2), J4.4 (GPIO2)
- net MUX_SEL_MCU: now reaches A1.1 (GPIO0), J4.1 (GPIO0)
- net MUX_SEL_MCU: now also R30.1, SW2.3 (C)
- net ~{DP_RST}: now reaches A1.2 (GPIO1), J4.2 (GPIO1)
- net VBUS_IN: now reaches A1.39 (VSYS), J10.19 (VSYS)
- net VBUS_IN: now also A1.40 (VBUS), J10.20 (VBUS)
- net at A1.TP2 (USB_DM): now also R33.2
- net at A1.TP3 (USB_DP): now also R31.2
- net MUX_SEL_PRE: no longer names the net of TP3.1, U1.2 (IN)
- net MUX_SEL_PRE: now also SW2.2 (B); no longer SW1.2 (B)
- new net MCU_USB_DN: R33.1
- new net MCU_USB_DP: R31.1
- new net MUX_SEL_MANUAL: SW1.2 (B), SW2.1 (A)
- no-connect marks 0 -> 1
Other:
- note added: "Pico 3V3 OUT (NC)"
- moved on the sheet: R7, R8, SW1, TP2, TP7

Commit message: Wire up more of the Pico
Parts:
- removed R31, R33: 27, Resistor_SMD:R_0603_1608Metric, symbol Device:R
- added R36: 10k, Resistor_SMD:R_0603_1608Metric, symbol Device:R
- A1: now not fitted; now left out of the parts list
Connections:
- net GND: now also J10.13 (AGND), J10.18 (GND), J10.3 (GND), J10.8 (GND), J4.13 (GND), J4.18 (GND), J4.3 (GND), J4.8 (GND), SW2.4 (A)
- net I2C_SCL: no longer A1.5 (GPIO3)
- net I2C_SDA: no longer A1.4 (GPIO2)
- net MUX_SEL_MCU: no longer A1.1 (GPIO0)
- net VBUS_IN: no longer A1.39 (VSYS), A1.40 (VBUS)
- net VCC_3.3V: now also R36.1
- net ~{DP_RST}: no longer A1.2 (GPIO1)
- net PI_RUN: now reaches SW2.5 (B)
- net PI_RUN: now also J10.10 (RUN)
- net at SW2.6 (C): now also R36.2
- net at J4.10 (GPIO7): no longer A1.10 (GPIO7)
- net at J4.11 (GPIO8): no longer A1.11 (GPIO8)
- net at J4.12 (GPIO9): no longer A1.12 (GPIO9)
- net at A1.13 (GND), A1.18 (GND), A1.23 (GND)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: no longer J10.18 (GND), J10.3 (GND), J10.8 (GND), J4.13 (GND), J4.18 (GND), J4.3 (GND), J4.8 (GND)
- net at J4.14 (GPIO10): no longer A1.14 (GPIO10)
- net at J4.15 (GPIO11): no longer A1.15 (GPIO11)
- net at J4.16 (GPIO12): no longer A1.16 (GPIO12)
- net at J4.17 (GPIO13): no longer A1.17 (GPIO13)
- net at J4.19 (GPIO14): no longer A1.19 (GPIO14)
- net at J4.20 (GPIO15): no longer A1.20 (GPIO15)
- net at J4.6 (GPIO4): no longer A1.6 (GPIO4)
- net at J4.7 (GPIO5): no longer A1.7 (GPIO5)
- net at J4.9 (GPIO6): no longer A1.9 (GPIO6)
- net at J10.1 (GPIO16): no longer A1.21 (GPIO16)
- net at A1.30 (RUN): no longer J10.10 (RUN)
- net at J10.11 (GPIO26_ADC0): no longer A1.31 (GPIO26_ADC0)
- net at J10.12 (GPIO27_ADC1): no longer A1.32 (GPIO27_ADC1)
- net at A1.33 (AGND): no longer J10.13 (AGND)
- net at J10.14 (GPIO28_ADC2): no longer A1.34 (GPIO28_ADC2)
- net at J10.15 (ADC_VREF): no longer A1.35 (ADC_VREF)
- net at J10.16 (3V3): no longer A1.36 (3V3)
- net at J10.17 (3V3_EN): no longer A1.37 (3V3_EN)
- net at J10.2 (GPIO17): no longer A1.22 (GPIO17)
- net at J10.4 (GPIO18): no longer A1.24 (GPIO18)
- net at J10.5 (GPIO19): no longer A1.25 (GPIO19)
- net at J10.6 (GPIO20): no longer A1.26 (GPIO20)
- net at J10.7 (GPIO21): no longer A1.27 (GPIO21)
- net at J10.9 (GPIO22): no longer A1.29 (GPIO22)
- no-connect marks 1 -> 27
Other:
- moved on the sheet: C88, C9, J10, J4, R13, R14, R17, R30, R32, R7, R8, SW1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
